Commit message: Move traquad to Isaac Sim 6.1 / Isaac Lab 3.0 and tune the rough task rewards
Track model and asset:
- track.xacro: track_model arg (rollers / cylinder with mimic joints), box track colliders, wheel_mu 0.75
- Isaac asset rebuilt: passive ankles, HFE Kd 10, 40 Nm per track, roller dry friction 0.06 Nm;
  cylinder variant in isaac_sim/assets/traquad_cylinder
- isaac_sim test scripts aligned to the current model; --roller_friction always applied,
  track_test.py --roller_friction, video_replica.py handles the cylinder model and logs a CSV
- sv_test.py (surface velocity test), README with the October 2026 findings

Isaac Lab 3.0 TraQuad tasks, now versioned in isaaclab_overlay/ and linked into an Isaac Lab
checkout by isaaclab_overlay/setup_isaaclab.sh:
- wheel action scale 66.7 rad/s (1 unit = 1 m/s of track), forward command limited to 0.5 m/s
- rewards: yaw tracking 1.0, action rate -0.01, HFE deviation -0.1, HFE torques -1e-3,
  ankle limits -5, wheel velocity difference -7.5e-4, new lateral velocity penalty -0.1,
  feet_air_time_stuck disabled (measured on single rollers, it penalized rotation in place)
- roller dry friction randomized per robot in 0.02-0.06 N m at startup
- gpu_max_num_partitions = 1 (PhysX GPU bug isaac-sim/IsaacLab#8121)

Co-Authored-By: Claude Opus 5.5 <noreply@anthropic.com>

File: src/mulinex_description/urdf/track.xacro (robot description, xacro)
@@ -2,4 +2,9 @@
 <robot xmlns:xacro="http://ros.org/wiki/xacro" name="track">
   <!-- ===================== ARGOMENTI COMUNI ===================== -->
+  <!-- track_model: "rollers" (default) = ground wheels with 8 passive rollers each;
+       "cylinder" = all wheels are plain primitive cylinders, wheels 1, 3, 4 follow wheel 2 through mimic joints
+       (one driven wheel per track, as the real belt). In both models the track body collides as a box -->
+  <xacro:arg name="track_model" default="rollers"/>
+  <xacro:property name="cylinder_tracks" value="${'$(arg track_model)' == 'cylinder'}"/>
   <!-- whole track (body + 4 wheels + rollers) = 1.0 kg x track_mass_scale = 0.325 kg (real robot);
        masses and inertias of body, wheels and rollers are scaled by the same factor -->
@@ -10,7 +15,8 @@
   <xacro:property name="wheel_izz" default="${1.15625e-05 * track_mass_scale}"/>
   <xacro:property name="wheel_mesh" default="file://$(find mulinex_description)/meshes//wheel.stl"/>
-  <!-- Wheel/roller contact. Isotropic friction (Isaac Sim default 0.5), lateral compliance
-       comes from passive rollers on the ground wheels: roller_damping tunes lateral resistance -->
-  <xacro:property name="wheel_mu" value="0.5"/>
+  <!-- Wheel/roller contact. Isotropic friction 0.75, the effective wheel-ground value of Isaac Sim
+       (open_traquad.py: ground 1.0 averaged with the robot default 0.5; the Gazebo ground keeps the SDF default 1.0,
+       the contact takes the minimum). Lateral compliance comes from passive rollers on the ground wheels -->
+  <xacro:property name="wheel_mu" value="0.75"/>
   <xacro:property name="roller_n" value="8"/>
   <xacro:property name="roller_radius" value="0.008"/>
@@ -83,5 +89,5 @@
   </xacro:macro>
   <!-- Macro RUOTA: rollers=true for ground wheels, false for the raised idler -->
-  <xacro:macro name="wheel" params="name parent xyz rpy rollers:=true">
+  <xacro:macro name="wheel" params="name parent xyz rpy rollers:=true mimic:=''">
     <link name="${name}">
       <xacro:if value="${rollers}">
@@ -122,4 +128,7 @@
       <axis xyz="0 0 1"/>
       <limit effort="10" velocity="100000"/>
+      <xacro:if value="${mimic != ''}">
+        <mimic joint="${mimic}" multiplier="1" offset="0"/>
+      </xacro:if>
     </joint>
     <xacro:if value="${rollers}">
@@ -164,8 +173,10 @@
         </material>
       </visual>
-      <collision>
-        <origin xyz="0 0 0" rpy="0 0 3.14159"/>
-        <geometry>
-          <mesh filename="${body_left_mesh}"/>
+      <!-- bounding box of body_left.stl (no convex hull of the mesh on steps and obstacles);
+           12.5 mm above the ground when the track lies flat, as the mesh -->
+      <collision>
+        <origin xyz="0.025 -0.0119 -0.0174" rpy="0 0 0"/>
+        <geometry>
+          <box size="0.05 0.1417 0.0869"/>
         </geometry>
       </collision>
@@ -206,8 +217,9 @@
         </material>
       </visual>
-      <collision>
-        <origin xyz="0 0 0" rpy="-1.5708 0 -3.14159"/>
-        <geometry>
-          <mesh filename="${body_right_mesh}"/>
+      <!-- bounding box of body_right.stl -->
+      <collision>
+        <origin xyz="-0.025 0.0174 -0.0119" rpy="0 0 0"/>
+        <geometry>
+          <box size="0.05 0.0869 0.1417"/>
         </geometry>
       </collision>
@@ -218,28 +230,28 @@
   <xacro:body_left name="body_left_H" parent="LH_UPPER_LEG"
                    xyz="-0.19 0.05 0" rpy="1.5708 0 1.5708" ankle_center="${-ankle_flat}"/>
-  <xacro:wheel name="wheel_1_LEFT_H" parent="body_left_H" xyz="0 0.0484063 -0.0583795" rpy="-6.12323e-17 -1.5708 0"/>
-  <xacro:wheel name="wheel_2_LEFT_H" parent="body_left_H" xyz="0 1.07779e-16 -0.0583795" rpy="-6.12323e-17 -1.5708 0"/>
-  <xacro:wheel name="wheel_3_LEFT_H" parent="body_left_H" xyz="0 -0.0510313 -0.0583795" rpy="-6.12323e-17 -1.5708 0"/>
-  <xacro:wheel name="wheel_4_LEFT_H" parent="body_left_H" xyz="0 -0.0766777 -0.0417374" rpy="-6.12323e-17 -1.5708 0" rollers="false"/>
+  <xacro:wheel name="wheel_1_LEFT_H" parent="body_left_H" xyz="0 0.0484063 -0.0583795" rpy="-6.12323e-17 -1.5708 0" rollers="${not cylinder_tracks}" mimic="${'joint_wheel_2_LEFT_H' if cylinder_tracks else ''}"/>
+  <xacro:wheel name="wheel_2_LEFT_H" parent="body_left_H" xyz="0 1.07779e-16 -0.0583795" rpy="-6.12323e-17 -1.5708 0" rollers="${not cylinder_tracks}"/>
+  <xacro:wheel name="wheel_3_LEFT_H" parent="body_left_H" xyz="0 -0.0510313 -0.0583795" rpy="-6.12323e-17 -1.5708 0" rollers="${not cylinder_tracks}" mimic="${'joint_wheel_2_LEFT_H' if cylinder_tracks else ''}"/>
+  <xacro:wheel name="wheel_4_LEFT_H" parent="body_left_H" xyz="0 -0.0766777 -0.0417374" rpy="-6.12323e-17 -1.5708 0" rollers="false" mimic="${'joint_wheel_2_LEFT_H' if cylinder_tracks else ''}"/>
   <!-- LEFT_F -->
   <xacro:body_left name="body_left_F" parent="LF_UPPER_LEG"
                    xyz="0.19 0.05 0" rpy="-1.5708 0 1.5708" ankle_center="${ankle_flat}"/>
-  <xacro:wheel name="wheel_1_LEFT_F" parent="body_left_F" xyz="0 0.0484063 -0.0583795" rpy="-6.12323e-17 -1.5708 0"/>
-  <xacro:wheel name="wheel_2_LEFT_F" parent="body_left_F" xyz="0 1.07779e-16 -0.0583795" rpy="-6.12323e-17 -1.5708 0"/>
-  <xacro:wheel name="wheel_3_LEFT_F" parent="body_left_F" xyz="0 -0.0510313 -0.0583795" rpy="-6.12323e-17 -1.5708 0"/>
-  <xacro:wheel name="wheel_4_LEFT_F" parent="body_left_F" xyz="0 -0.0766777 -0.0417374" rpy="-6.12323e-17 -1.5708 0" rollers="false"/>
+  <xacro:wheel name="wheel_1_LEFT_F" parent="body_left_F" xyz="0 0.0484063 -0.0583795" rpy="-6.12323e-17 -1.5708 0" rollers="${not cylinder_tracks}" mimic="${'joint_wheel_2_LEFT_F' if cylinder_tracks else ''}"/>
+  <xacro:wheel name="wheel_2_LEFT_F" parent="body_left_F" xyz="0 1.07779e-16 -0.0583795" rpy="-6.12323e-17 -1.5708 0" rollers="${not cylinder_tracks}"/>
+  <xacro:wheel name="wheel_3_LEFT_F" parent="body_left_F" xyz="0 -0.0510313 -0.0583795" rpy="-6.12323e-17 -1.5708 0" rollers="${not cylinder_tracks}" mimic="${'joint_wheel_2_LEFT_F' if cylinder_tracks else ''}"/>
+  <xacro:wheel name="wheel_4_LEFT_F" parent="body_left_F" xyz="0 -0.0766777 -0.0417374" rpy="-6.12323e-17 -1.5708 0" rollers="false" mimic="${'joint_wheel_2_LEFT_F' if cylinder_tracks else ''}"/>
   <!-- RIGHT_F -->
   <xacro:body_right name="body_right_F" parent="RF_UPPER_LEG"
                     xyz="0.19 -0.05 0" rpy="3.14159 0 1.5708" ankle_center="${ankle_flat}"/>
-  <xacro:wheel name="wheel_1_RIGHT_F" parent="body_right_F" xyz="2.08167e-17 0.0583795 0.0484062" rpy="-1.5708 0 -1.5708"/>
-  <xacro:wheel name="wheel_2_RIGHT_F" parent="body_right_F" xyz="0 0.0583795 1.10544e-16" rpy="-1.5708 0 -1.5708"/>
-  <xacro:wheel name="wheel_3_RIGHT_F" parent="body_right_F" xyz="-2.08167e-17 0.0583795 -0.0510312" rpy="-1.5708 0 -1.5708"/>
-  <xacro:wheel name="wheel_4_RIGHT_F" parent="body_right_F" xyz="-3.46945e-17 0.0417374 -0.0766777" rpy="-1.5708 0 -1.5708" rollers="false"/>
+  <xacro:wheel name="wheel_1_RIGHT_F" parent="body_right_F" xyz="2.08167e-17 0.0583795 0.0484062" rpy="-1.5708 0 -1.5708" rollers="${not cylinder_tracks}" mimic="${'joint_wheel_2_RIGHT_F' if cylinder_tracks else ''}"/>
+  <xacro:wheel name="wheel_2_RIGHT_F" parent="body_right_F" xyz="0 0.0583795 1.10544e-16" rpy="-1.5708 0 -1.5708" rollers="${not cylinder_tracks}"/>
+  <xacro:wheel name="wheel_3_RIGHT_F" parent="body_right_F" xyz="-2.08167e-17 0.0583795 -0.0510312" rpy="-1.5708 0 -1.5708" rollers="${not cylinder_tracks}" mimic="${'joint_wheel_2_RIGHT_F' if cylinder_tracks else ''}"/>
+  <xacro:wheel name="wheel_4_RIGHT_F" parent="body_right_F" xyz="-3.46945e-17 0.0417374 -0.0766777" rpy="-1.5708 0 -1.5708" rollers="false" mimic="${'joint_wheel_2_RIGHT_F' if cylinder_tracks else ''}"/>
   <!-- RIGHT_H -->
   <xacro:body_right name="body_right_H" parent="RH_UPPER_LEG"
                     xyz="-0.19 -0.05 0" rpy="0 0 1.5708" ankle_center="${-ankle_flat}"/>
-  <xacro:wheel name="wheel_1_RIGHT_H" parent="body_right_H" xyz="2.08167e-17 0.0583795 0.0484062" rpy="-1.5708 0 -1.5708"/>
-  <xacro:wheel name="wheel_2_RIGHT_H" parent="body_right_H" xyz="0 0.0583795 1.10544e-16" rpy="-1.5708 0 -1.5708"/>
-  <xacro:wheel name="wheel_3_RIGHT_H" parent="body_right_H" xyz="-2.08167e-17 0.0583795 -0.0510312" rpy="-1.5708 0 -1.5708"/>
-  <xacro:wheel name="wheel_4_RIGHT_H" parent="body_right_H" xyz="-3.46945e-17 0.0417374 -0.0766777" rpy="-1.5708 0 -1.5708" rollers="false"/>
+  <xacro:wheel name="wheel_1_RIGHT_H" parent="body_right_H" xyz="2.08167e-17 0.0583795 0.0484062" rpy="-1.5708 0 -1.5708" rollers="${not cylinder_tracks}" mimic="${'joint_wheel_2_RIGHT_H' if cylinder_tracks else ''}"/>
+  <xacro:wheel name="wheel_2_RIGHT_H" parent="body_right_H" xyz="0 0.0583795 1.10544e-16" rpy="-1.5708 0 -1.5708" rollers="${not cylinder_tracks}"/>
+  <xacro:wheel name="wheel_3_RIGHT_H" parent="body_right_H" xyz="-2.08167e-17 0.0583795 -0.0510312" rpy="-1.5708 0 -1.5708" rollers="${not cylinder_tracks}" mimic="${'joint_wheel_2_RIGHT_H' if cylinder_tracks else ''}"/>
+  <xacro:wheel name="wheel_4_RIGHT_H" parent="body_right_H" xyz="-3.46945e-17 0.0417374 -0.0766777" rpy="-1.5708 0 -1.5708" rollers="false" mimic="${'joint_wheel_2_RIGHT_H' if cylinder_tracks else ''}"/>
 </robot>

Commit message: TraQuad: ankle driven by the sprocket in the air, default stance 1.47, final motor limits
Track and ankle model:
- the drive sprocket is coaxial with the ankle: the ankle is passive on the ground (damping
  0.01 N m s/rad) and, after 50 ms without contact, a PI velocity controller turns the frame at
  v_track / r_sprocket until its end stop (Kp 0.2, Ki 2, max 0.05 N m, anti-windup). In Isaac Lab
  the track action drives it from the contact sensor (not a policy output); isaac_sim/ankle_control.py
  and open_traquad.py implement the same law
- track CoM below the ankle axis with the track flat; ankle end stops +-30 deg around the flat pose
  of the default stance, relative to the upper leg
- default stance HFE +-1.47 (hips hold the robot with ~1.5 N m instead of 3.2-3.6 at 1.13)
- hip limit 10 N m (was 5, saturated in training); track motor 1.5 N m per track (was 40: torque
  spikes tipped the tracks onto their stops in turns)

Training: ankle end-stop penalty off, track_air_time_stuck weight 1.0, ground friction 0.3-0.8
(tracks tip above ~0.85 with this sprocket radius).

Tools: ankle_swing.py (suspended robot, track speed sequences, video), track_test.py --hfe,
--no_coupling, --ankle_range and leg/ankle/motor metrics; README with the findings.

Co-Authored-By: Claude Opus 5.5 <noreply@anthropic.com>

File: src/mulinex_description/urdf/track.xacro (robot description, xacro)
@@ -28,9 +28,12 @@
   <xacro:property name="roller_inertia" value="1e-5"/>
   <xacro:property name="body_mass" value="${0.6 * track_mass_scale}"/>
-  <!-- Passive ankle: range centred on the pose where the track lies flat
-       (wheels 1-3 level) with HFE at init_pos (+-1.13 rad) -->
-  <xacro:property name="ankle_flat" value="0.441"/>
-  <xacro:property name="ankle_range" value="0.35"/>
-  <xacro:property name="ankle_damping" value="0.05"/>
+  <!-- Ankle end stops (relative to the upper leg): +-30 deg around the pose where the track lies flat
+       (wheels 1-3 level) in the default stance, HFE +-1.47 rad: ankle_flat = pi/2 - 1.47 -->
+  <xacro:property name="ankle_flat" value="0.1008"/>
+  <xacro:property name="ankle_range" value="0.5236"/>
+  <!-- passive ankle damping: a hanging track is a damped pendulum, k = m g d = 0.077 N m/rad (d = 24 mm),
+       I = 1.17e-3 kg m2 about the ankle (rollers' armature-like inertia included): 1.3 Hz, damping ratio 0.5.
+       In Isaac the ankle is also velocity controlled when the track is in the air (drive sprocket coaxial with it) -->
+  <xacro:property name="ankle_damping" value="0.01"/>
   <xacro:property name="body_left_mesh" default="file://$(find mulinex_description)/meshes//body_left.stl"/>
   <xacro:property name="body_right_mesh" default="file://$(find mulinex_description)/meshes//body_right.stl"/>
@@ -151,5 +154,7 @@
     <link name="${name}">
       <inertial>
-        <origin xyz="0.0238777 -0.00119624 -0.00412068" rpy="0 0 0"/>
+        <!-- along the track (y) the CoM is placed so that the whole track (body + 4 wheels) has its CoM straight
+             below the ankle axis when the track is flat: a hanging track swings about the flat pose -->
+        <origin xyz="0.0238777 0.0132172 -0.00412068" rpy="0 0 0"/>
         <mass value="${body_mass}"/>
         <inertia ixx="${0.000408384 * track_mass_scale}" ixy="${6.93353e-06 * track_mass_scale}" ixz="${3.09979e-05 * track_mass_scale}"
@@ -195,5 +200,6 @@
     <link name="${name}">
       <inertial>
-        <origin xyz="-0.0238777 0.00412068 -0.00119624" rpy="0 0 0"/>
+        <!-- mirror of body_left: along the track (z) CoM below the ankle axis with the track flat -->
+        <origin xyz="-0.0238777 0.00412068 0.0132172" rpy="0 0 0"/>
         <mass value="${body_mass}"/>
         <inertia ixx="${0.000408384 * track_mass_scale}" ixy="${3.09979e-05 * track_mass_scale}" ixz="${-6.93353e-06 * track_mass_scale}"
